File: PIC18.kicad_sch (KiCad schematic)
At the start: 32 parts, among them J1 Conn_02x20_Counter_Clockwise, J2 Conn_01x06, J3 USB_A, J4 Conn_01x03, J5 Conn_01x02, J6 Conn_01x02, J7 Conn_01x08, J8 USB_OTG, U1 PIC18F4620, U2 LM4040DBZ-4.1, U3 FT230XS, Y1 8 MHz

Commit message: Updates
Parts:
- removed J7: Conn_01x08, Connector_PinHeader_2.54mm:PinHeader_2x04_P2.54mm_Vertical, symbol Connector_Generic:Conn_01x08
- removed J8: USB_OTG, Connector_USB:USB_Mini-B_Lumberg_2486_01_Horizontal, symbol Connector:USB_OTG
- added D4, D5, D6, D7: D_Zener, ZM4748A_L0G:DIOMELF5124N, symbol Device:D_Zener
- added D8: ZMM5V1, ZM4748A_L0G:DIOMELF5124N, symbol Device:D_Zener
- added H1, H2, H3, H4: MountingHole_Pad, MountingHole:MountingHole_4.3mm_M4_ISO14580_Pad_TopBottom, symbol Mechanical:MountingHole_Pad
- added J10: Port B, PinHeaders:PinHeader_2x04_P2.54mm_Vertical_Yellow, symbol Connector_Generic:Conn_01x08
- added J11: Port C, PinHeaders:PinHeader_2x04_P2.54mm_Vertical_Blue, symbol Connector_Generic:Conn_01x08
- added J12: Port D, PinHeaders:PinHeader_2x04_P2.54mm_Vertical_White, symbol Connector_Generic:Conn_01x08
- added J13, J14: Conn_01x03, Connector_PinHeader_2.54mm:PinHeader_1x03_P2.54mm_Vertical, symbol Connector_Generic:Conn_01x03
- added J7: USB_OTG, Connector_USB:USB_Mini-B_Lumberg_2486_01_Horizontal, symbol Connector:USB_OTG
- added J8: Port A, PinHeaders:PinHeader_2x04_P2.54mm_Vertical_Red, symbol Connector_Generic:Conn_01x08
- added J9: Port E, PinHeaders:PinHeader_2x04_P2.54mm_Vertical_Green, symbol Connector_Generic:Conn_01x08
- added R10, R11, R12, R13, R14, R19, R20, R21, R7, R8, R9: 220, Resistor_SMD:R_0402_1005Metric, symbol Device:R_US
- added R15: 100, Resistor_SMD:R_0402_1005Metric, symbol Device:R_US
- added R16: 1k, Resistor_SMD:R_0402_1005Metric, symbol Device:R_US
- added R17: 10k, Resistor_SMD:R_0402_1005Metric, symbol Device:R_US
- added R18: 100k, Resistor_SMD:R_0402_1005Metric, symbol Device:R_US
- added RN2, RN3, RN4, RN5, RN6, RN7: 220, Resistor_SMD:R_Array_Convex_4x0603, symbol Device:R_Pack04
- RN1: value R_Pack04 -> 220
Connections:
- net GND: now also D3.2 (A), D4.2 (A), D5.2 (A), D6.2 (A), D7.2 (A), D8.2 (A), H1.1, H2.1, H3.1, H4.1, J13.2 (Pin_2), J7.5 (GND), J7.6 (Shield)
- net OSC1/CLKI/RA7: now also R13.1
- net OSC2/CLKO/RA6: now also R14.1
- net RA0/AN0: now also D3.1 (K), R7.1
- net RA1/AN1: now also D4.1 (K), R8.1
- net RA2/AN2/VREF-/CVREF: now also D5.1 (K), R9.1
- net RA3/AN3/VREF+: now also D6.1 (K), J9.4 (Pin_4), R10.1, R15.1, R16.1, R17.1, R18.1
- net RA4/T0CKI/C1OUT: now also D7.1 (K), R11.1
- net RA5/AN4/SS*/HLVDIN/C2OUT: now also J1.7 (Pin_7), D8.1 (K), R12.1
- net RC3/SCK/SCL: now also RN4.8 (R1.2)
- net RD0/PSP0: now also RN6.5 (R4.2)
- net RD1/PSP1: now also RN6.6 (R3.2)
- net RD5/PSP5/P1B: now also RN7.6 (R3.2)
- net RD6/PSP6/P1C: now also RN7.7 (R2.2)
- net RD7/PSP7/P1D: now also RN7.8 (R1.2)
- net RE0/RD*/AN5: now also RN1.5 (R4.2)
- net RE1/WR*/AN6: now also RN1.6 (R3.2)
- net RE2/CS*/AN7: now also RN1.7 (R2.2)
- net VCC: now also J7.1 (VBUS)
- net at J3.2 (D-), R3.1: now also J7.2 (D-)
- net at J3.3 (D+), R2.1: now also J7.3 (D+)
- net at RN1.2 (R2.1): now also J9.3 (Pin_3)
- net at RN1.3 (R3.1): now also J9.2 (Pin_2)
- net at RN1.4 (R4.1): now also J9.1 (Pin_1)
- new net: J8.7 (Pin_7), R13.2
- new net: J9.8 (Pin_8), R18.2
- new net: J10.1 (Pin_1), RN2.4 (R4.1)
- new net: J10.2 (Pin_2), RN2.3 (R3.1)
- new net: J10.3 (Pin_3), RN2.2 (R2.1)
- new net: J10.4 (Pin_4), RN2.1 (R1.1)
- new net: J10.5 (Pin_5), RN3.4 (R4.1)
- new net: J10.6 (Pin_6), RN3.3 (R3.1)
- new net: J10.7 (Pin_7), RN3.2 (R2.1)
- new net: J10.8 (Pin_8), RN3.1 (R1.1)
- new net: J11.8 (Pin_8), RN5.1 (R1.1)
- new net: J11.7 (Pin_7), RN5.2 (R2.1)
- new net: J11.6 (Pin_6), RN5.3 (R3.1)
- new net: J11.5 (Pin_5), RN5.4 (R4.1)
- new net: J14.3 (Pin_3), R21.2
- new net: J14.2 (Pin_2), R20.2
- new net: J8.6 (Pin_6), R12.2
- new net: J9.7 (Pin_7), R17.2
- new net: J8.4 (Pin_4), R10.2
- new net: J9.6 (Pin_6), R16.2
- new net: J8.2 (Pin_2), R8.2
- new net: J9.5 (Pin_5), R15.2
- new net: J8.1 (Pin_1), R7.2
- new net: J12.8 (Pin_8), RN7.1 (R1.1)
- new net: J12.7 (Pin_7), RN7.2 (R2.1)
- new net: J12.6 (Pin_6), RN7.3 (R3.1)
- new net: J12.5 (Pin_5), RN7.4 (R4.1)
- new net: J14.1 (Pin_1), R19.2
- new net: J8.5 (Pin_5), R11.2
- new net: J8.3 (Pin_3), R9.2
- new net: J12.4 (Pin_4), RN6.1 (R1.1)
- new net: J12.3 (Pin_3), RN6.2 (R2.1)
- new net: J12.2 (Pin_2), RN6.3 (R3.1)
- new net: J12.1 (Pin_1), RN6.4 (R4.1)
- new net: J11.4 (Pin_4), RN4.1 (R1.1)
- new net: J11.3 (Pin_3), RN4.2 (R2.1)
- new net: J11.2 (Pin_2), RN4.3 (R3.1)
- new net: J11.1 (Pin_1), RN4.4 (R4.1)
- new net: J8.8 (Pin_8), R14.2
- new net RB0/INT0/FLT0/AN12: RN3.8 (R1.2)
- new net RB1/INT1/AN10: RN3.7 (R2.2)
- new net RB2/INT2/AN8: RN3.6 (R3.2)
- new net RB3/AN9/CCP2(1): RN3.5 (R4.2)
- new net RB4/KBI0/AN11: RN2.8 (R1.2)
- new net RB5/KBI1/PGM: RN2.7 (R2.2)
- new net RB6/KBI2/PGC: RN2.6 (R3.2)
- new net RB7/KBI3/PGD: RN2.5 (R4.2)
- new net RC0/T1OSO/T13CKI: RN4.5 (R4.2)
- new net RC1/T1OSI/CCP2(1): RN4.6 (R3.2)
- new net RC2/CCP1/P1A: RN4.7 (R2.2)
- new net RC4/SDI/SDA: R21.1, RN5.5 (R4.2)
- new net RC5/SDO: R20.1, RN5.6 (R3.2)
- new net RC6/TX/CK: J13.3 (Pin_3), R19.1, RN5.7 (R2.2)
- new net RC7/RX/DT: RN5.8 (R1.2)
- new net RD2/PSP2: RN6.7 (R2.2)
- new net RD3/PSP3: RN6.8 (R1.2)
- new net RD4/PSP4: RN7.5 (R4.2)
- no-connect marks 2 -> 5
Other:
- moved on the sheet: D3, J1, RN1
