File: PIC18.kicad_sch (KiCad schematic)
At the start: 68 parts, among them J1 Conn_02x20_Odd_Even, J10 Port B, J11 Port C, J12 Port D, J13 Conn_01x03, J14 Conn_01x03, J2 Conn_01x06, J3 USB_A, J4 Conn_01x03, J5 Conn_01x02, J6 Conn_01x02, J7 USB_OTG, J8 Port A, J9 Port E, U1 PIC18F4620, U2 LM4040DBZ-4.1, U3 FT230XS, Y1 8 MHz

Commit message: Updated schematic
Connections:
- net GND: now also J1.31 (Pin_31); no longer J13.2 (Pin_2)
- net OSC2/CLKO/RA6: now also J1.14 (Pin_14)
- net RB0/INT0/FLT0/AN12: now also J1.33 (Pin_33)
- net RB2/INT2/AN8: now also J1.35 (Pin_35)
- net RB4/KBI0/AN11: now also J1.37 (Pin_37)
- net RB6/KBI2/PGC: now also J1.39 (Pin_39)
- net RC1/T1OSI/CCP2(1): now also J1.16 (Pin_16)
- net RC3/SCK/SCL: now also J1.18 (Pin_18)
- net RC4/SDI/SDA: now also J1.23 (Pin_23)
- net RC6/TX/CK: now also J1.25 (Pin_25)
- net RD1/PSP1: now also J1.20 (Pin_20)
- net RD2/PSP2: now also J1.21 (Pin_21)
- net RD4/PSP4: now also J1.27 (Pin_27)
- net RD6/PSP6/P1C: now also J1.29 (Pin_29)
Changed lines of the file:
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@@
 	(wire
 		(pts
-			(xy 311.15 35.56) (xy 311.15 40.64)
-		)
-		(stroke
-			(width 0)
-			(type default)
-		)
-	)
-	(wire
-		(pts
 			(xy 129.54 132.08) (xy 143.51 132.08)
 		)
@@
 	(wire
 		(pts
-			(xy 312.42 35.56) (xy 311.15 35.56)
-		)
-		(stroke
-			(width 0)
-			(type default)
-		)
-	)
-	(wire
-		(pts
 			(xy 93.98 76.2) (xy 96.52 76.2)
 		)
@@
 		)
 	)
+	(label "RD6/PSP6/P1C"
+		(at 199.39 250.19 180)
+		(fields_autoplaced yes)
+		(effects
+			(font
+				(size 1.27 1.27)
+			)
+			(justify right bottom)
+		)
+	)
 	(label "VDD"
 		(at 199.39 227.33 180)
@@
 		)
 	)
+	(label "RD4/PSP4"
+		(at 199.39 247.65 180)
+		(fields_autoplaced yes)
+		(effects
+			(font
+				(size 1.27 1.27)
+			)
+			(justify right bottom)
+		)
+	)
 	(label "RC6{slash}TX{slash}CK"
 		(at 259.08 138.43 180)
@@
 		)
 	)
+	(label "VSS"
+		(at 199.39 252.73 180)
+		(fields_autoplaced yes)
+		(effects
+			(font
+				(size 1.27 1.27)
+			)
+			(justify right bottom)
+		)
+	)
 	(label "RB5/KBI1/PGM"
 		(at 214.63 260.35 0)
@@
 		)
 	)
+	(label "OSC2/CLKO/RA6"
+		(at 214.63 229.87 0)
+		(fields_autoplaced yes)
+		(effects
+			(font
+				(size 1.27 1.27)
+			)
+			(justify left bottom)
+		)
+	)
 	(label "*MCLR/VPP/RE3"
 		(at 50.8 38.1 180)
@@
 		)
 	)
+	(label "RD2/PSP2"
+		(at 199.39 240.03 180)
+		(fields_autoplaced yes)
+		(effects
+			(font
+				(size 1.27 1.27)
+			)
+			(justify right bottom)
+		)
+	)
 	(label "RC4{slash}SDI{slash}SDA"
 		(at 299.72 60.96 180)
@@
 		)
 	)
+	(label "RC3/SCK/SCL"
+		(at 214.63 234.95 0)
+		(fields_autoplaced yes)
+		(effects
+			(font
+				(size 1.27 1.27)
+			)
+			(justify left bottom)
+		)
+	)
 	(label "RD5/PSP5/P1B"
 		(at 137.16 243.84 0)
@@
 		)
 	)
+	(label "RC4/SDI/SDA"
+		(at 199.39 242.57 180)
+		(fields_autoplaced yes)
+		(effects
+			(font
+				(size 1.27 1.27)
+			)
+			(justify right bottom)
+		)
+	)
 	(label "*MCLR/VPP/RE3"
 		(at 67.31 213.36 180)
@@
 		)
 	)
+	(label "RB6/KBI2/PGC"
+		(at 199.39 262.89 180)
+		(fields_autoplaced yes)
+		(effects
+			(font
+				(size 1.27 1.27)
+			)
+			(justify right bottom)
+		)
+	)
 	(label "RD3{slash}PSP3"
 		(at 321.31 133.35 180)
@@
 	)
 	(label "VDD"
-		(at 215.9 252.73 0)
+		(at 214.63 252.73 0)
 		(fields_autoplaced yes)
 		(effects
@@
 		)
 	)
+	(label "RC6/TX/CK"
+		(at 199.39 245.11 180)
+		(fields_autoplaced yes)
+		(effects
+			(font
+				(size 1.27 1.27)
+			)
+			(justify right bottom)
+		)
+	)
 	(label "RD4{slash}PSP4"
 		(at 321.31 135.89 180)
@@
 		)
 	)
+	(label "RC1/T1OSI/CCP2(1)"
+		(at 214.63 232.41 0)
+		(fields_autoplaced yes)
+		(effects
+			(font
+				(size 1.27 1.27)
+			)
+			(justify left bottom)
+		)
+	)
 	(label "RC5/SDO"
 		(at 137.16 254 0)
@@
 		)
 	)
+	(label "RD1/PSP1"
+		(at 214.63 237.49 0)
+		(fields_autoplaced yes)
+		(effects
+			(font
+				(size 1.27 1.27)
+			)
+			(justify left bottom)
+		)
+	)
 	(label "RA5/AN4/SS*/HLVDIN/C2OUT"
 		(at 199.39 222.25 180)
@@
 	)
 	(label "VSS"
-		(at 215.9 227.33 0)
+		(at 214.63 227.33 0)
 		(fields_autoplaced yes)
 		(effects
@@
 		)
 	)
+	(label "RB4/KBI0/AN11"
+		(at 199.39 260.35 180)
+		(fields_autoplaced yes)
+		(effects
+			(font
+				(size 1.27 1.27)
+			)
+			(justify right bottom)
+		)
+	)
 	(label "RC7/RX/DT"
 		(at 154.94 31.75 0)
@@
 		)
 	)
+	(label "RB0/INT0/FLT0/AN12"
+		(at 199.39 255.27 180)
+		(fields_autoplaced yes)
+		(effects
+			(font
+				(size 1.27 1.27)
+			)
+			(justify right bottom)
+		)
+	)
 	(label "RC2/CCP1/P1A"
 		(at 199.39 234.95 180)
@@
 		)
 	)
+	(label "RB2/INT2/AN8"
+		(at 199.39 257.81 180)
+		(fields_autoplaced yes)
+		(effects
+			(font
+				(size 1.27 1.27)
+			)
+			(justify right bottom)
+		)
+	)
 	(symbol
 		(lib_id "Device:R_US")
@@
 					(unit 1)
 				)
-			)
-		)
-	)
-	(symbol
-		(lib_id "power:GND")
-		(at 311.15 40.64 0)
-		(unit 1)
-		(exclude_from_sim no)
-		(in_bom yes)
-		(on_board yes)
-		(dnp no)
-		(fields_autoplaced yes)
-		(property "Reference" "#PWR026"
-			(at 311.15 46.99 0)
-			(effects
-				(font
-					(size 1.27 1.27)
-				)
-				(hide yes)
-			)
-		)
-		(property "Value" "GND"
-			(at 311.15 45.72 0)
-			(effects
-				(font
-					(size 1.27 1.27)
-				)
-			)
-		)
-		(property "Footprint" ""
-			(at 311.15 40.64 0)
-			(effects
-				(font
-					(size 1.27 1.27)
-				)
-				(hide yes)
-			)
-		)
-		(property "Datasheet" ""
-			(at 311.15 40.64 0)
-			(effects
-				(font
-					(size 1.27 1.27)
-				)
-				(hide yes)
-			)
-		)
-		(property "Description" "Power symbol creates a global label with name \"GND\" , ground"
-			(at 311.15 40.64 0)
-			(effects
-				(font
-					(size 1.27 1.27)
-				)
-				(hide yes)
-			)
-		)
-		(pin "1"
-		)
-		(instances
-			(project "PIC18"
-				(path "/e4a6b067-3b9b-4409-bea0-0b6131f207b6"
-					(reference "#PWR026")
-					(unit 1)
-				)
