File: _autosave-PIC18.kicad_sch (KiCad schematic)
At the start: 75 parts, among them J1 Conn_02x20_Odd_Even, J10 Port B, J11 Port C, J12 Port D, J13 Conn_01x03, J14 Conn_01x03, J15 Conn_01x03, J16 Conn_01x03, J2 Conn_01x06, J3 USB_A, J4 Conn_01x03, J5 Conn_01x02, J6 Conn_01x02, J7 USB_OTG, J8 Port A, J9 Port E, U1 PIC18F4620, U2 LM4040DBZ-4.1, U3 FT230XS, Y1 8 MHz

Commit message: lots of changes
Parts:
- C6: value 100n -> 100nF
Changed lines of the file:
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@@
 			)
 		)
-		(property "Value" "100n"
+		(property "Value" "100nF"
 			(at 130.048 110.998 90)
 			(effects
