File: PIC18.kicad_pcb (KiCad board)
At the start: 2 copper layers, 80 x 80 mm, 75 parts, among them J1 Conn_02x20_Odd_Even, J10 Port B, J11 Port C, J12 Port D, J13 Conn_01x03, J14 Conn_01x03, J15 Conn_01x03, J16 Conn_01x03, J2 Conn_01x06, J3 USB_A, J4 Conn_01x03, J5 Conn_01x02, J6 Conn_01x02, J7 USB_OTG, J8 Port A, J9 Port E, U1 PIC18F4620, U2 LM4040DBZ-4.1, U3 FT230XS, Y1 8 MHz

Commit message: Routing
Parts:
- C6: value 100n -> 100nF
- moved R11 23.0 mm to (165.4, 81.0)
- moved R12 22.5 mm to (165.4, 82.0)
- moved R13 22.1 mm to (165.4, 83.0)
- moved R14 21.7 mm to (165.4, 84.0)
- moved D3 21.2 mm to (155.2, 69.0), turned to 0 degrees
- moved D8 10.9 mm to (155.2, 76.1), turned to 0 degrees
- moved D6 7.09 mm to (138.5, 76.1)
- moved C8 6.56 mm to (112.2, 129.0), turned to -90 degrees
- moved D7 5.50 mm to (155.2, 72.6), turned to 0 degrees
- moved H4 5.48 mm to (172.8, 138.0)
- moved J1 5.41 mm to (145.6, 69.0)
- moved D4 5.10 mm to (138.5, 72.6)
- moved R10 5.03 mm to (165.4, 77.4)
- moved R9 4.39 mm to (165.4, 76.4)
- moved D5 4.27 mm to (138.5, 69.1)
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Connections:
- J13 pad 1: unconnected-(J13-Pin_1-Pad1) -> GND
- J4 pad 2: /RA1/AN1 -> /VREF+
- J4 pad 3: /RA3/AN3/VREF+ -> Net-(J4-Pin_3)
- J7 pad 1: VCC -> Net-(J3-VBUS)
- J9 pad 4: /RA3/AN3/VREF+ -> /VREF+
- R15 pad 1: /RA3/AN3/VREF+ -> /VREF+
- R16 pad 1: /RA3/AN3/VREF+ -> /VREF+
- R17 pad 1: /RA3/AN3/VREF+ -> /VREF+
- R18 pad 1: /RA3/AN3/VREF+ -> /VREF+
- R5 pad 2: /RA3/AN3/VREF+ -> Net-(J4-Pin_3)
- R6 pad 2: /RA3/AN3/VREF+ -> Net-(J4-Pin_3)
- U2 pad 1: /RA3/AN3/VREF+ -> Net-(J4-Pin_3)
Routing:
- net GND: track 0.00 -> 53.8 mm, vias 0 -> 13
- net /OSC1/CLKI/RA7: track 0.00 -> 52.8 mm, vias 0 -> 1
- net Net-(J3-VBUS): track 0.00 -> 39.0 mm, vias 0 -> 2
- net /OSC2/CLKO/RA6: track 0.00 -> 38.4 mm, vias 0 -> 1
- net /RB1/INT1/AN10: track 0.00 -> 37.8 mm
- net /RB0/INT0/FLT0/AN12: track 0.00 -> 36.7 mm
- net /RC6/TX/CK: track 0.00 -> 33.4 mm, vias 0 -> 1
- net Net-(J3-D+): track 0.00 -> 29.7 mm, vias 0 -> 2
- net Net-(J3-D-): track 0.00 -> 29.5 mm
- net /RD0/PSP0: track 0.00 -> 28.7 mm
- net /RB5/KBI1/PGM: track 0.00 -> 28.6 mm
- net /RC7/RX/DT: track 0.00 -> 28.4 mm, vias 0 -> 1
- net /RD2/PSP2: track 0.00 -> 28.2 mm
- net /RA3/AN3/VREF+: track 0.00 -> 28.0 mm, vias 0 -> 1
- net /RD1/PSP1: track 0.00 -> 27.4 mm, vias 0 -> 1
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- added copper zone on B.Cu, net GND
- added copper zone on F.Cu, net VCC
Other:
- board size 80 x 80 mm -> 76.6 x 75.6 mm

Commit message: Placement
Routing:
- net /RB1/INT1/AN10: track 37.8 -> 0.00 mm
- net /RB0/INT0/FLT0/AN12: track 36.7 -> 0.00 mm
- net /RC6/TX/CK: track 33.4 -> 0.00 mm, vias 1 -> 0
- net /RD0/PSP0: track 28.7 -> 0.00 mm
- net /RB5/KBI1/PGM: track 28.6 -> 0.00 mm
- net /RC7/RX/DT: track 28.4 -> 0.00 mm, vias 1 -> 0
- net /RD2/PSP2: track 28.2 -> 0.00 mm
- net /RA3/AN3/VREF+: track 28.0 -> 0.00 mm, vias 1 -> 0
- net /RD1/PSP1: track 27.4 -> 0.00 mm, vias 1 -> 0
- net /RB4/KBI0/AN11: track 27.4 -> 0.00 mm
- net /RA2/AN2/VREF-/CVREF: track 27.0 -> 0.00 mm, vias 1 -> 0
- net /RA1/AN1: track 26.9 -> 0.00 mm, vias 1 -> 0
- net /RB2/INT2/AN8: track 26.7 -> 0.00 mm, vias 1 -> 0
- net /RD3/PSP3: track 26.5 -> 0.00 mm, vias 1 -> 0
- net /RD4/PSP4: track 25.7 -> 0.00 mm
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
Commit message: Schematic edit
Changed lines of the file:
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@@
 	)
 	(segment
-		(start 110 74.24)
+		(start 111 77.75)
 		(end 110 77.75)
 		(width 0.2)
@@
 	)
 	(segment
-		(start 111 77.75)
-		(end 110 77.75)
+		(start 110 77.75)
+		(end 110 74.24)
 		(width 0.2)
 		(layer "F.Cu")

Commit message: Silkscreen edits
Other:
- copper layers 2 -> 4
Changed lines of the file:
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@@
 	(layers
 		(0 "F.Cu" signal)
+		(1 "In1.Cu" signal)
+		(2 "In2.Cu" signal)
 		(31 "B.Cu" signal)
 		(32 "B.Adhes" user "B.Adhesive")
@@
 	)
 	(setup
+		(stackup
+			(layer "F.SilkS"
+				(type "Top Silk Screen")
+			)
+			(layer "F.Paste"
+				(type "Top Solder Paste")
+			)
+			(layer "F.Mask"
+				(type "Top Solder Mask")
+				(thickness 0.01)
+			)
+			(layer "F.Cu"
+				(type "copper")
+				(thickness 0.035)
+			)
+			(layer "dielectric 1"
+				(type "prepreg")
+				(thickness 0.1)
+				(material "FR4")
+				(epsilon_r 4.5)
+				(loss_tangent 0.02)
+			)
+			(layer "In1.Cu"
+				(type "copper")
+				(thickness 0.035)
+			)
+			(layer "dielectric 2"
+				(type "core")
+				(thickness 1.24)
+				(material "FR4")
+				(epsilon_r 4.5)
+				(loss_tangent 0.02)
+			)
+			(layer "In2.Cu"
+				(type "copper")
+				(thickness 0.035)
+			)
+			(layer "dielectric 3"
+				(type "prepreg")
+				(thickness 0.1)
+				(material "FR4")
+				(epsilon_r 4.5)
+				(loss_tangent 0.02)
+			)
+			(layer "B.Cu"
+				(type "copper")
+				(thickness 0.035)
+			)
+			(layer "B.Mask"
+				(type "Bottom Solder Mask")
+				(thickness 0.01)
+			)
+			(layer "B.Paste"
+				(type "Bottom Solder Paste")
+			)
+			(layer "B.SilkS"
+				(type "Bottom Silk Screen")
+			)
+			(copper_finish "None")
+			(dielectric_constraints no)
+		)
 		(pad_to_mask_clearance 0)
 		(allow_soldermask_bridges_in_footprints no)
@@
 		(tags "mounting hole 4.3mm m4 iso14580")
 		(property "Reference" "H4"
-			(at 0 -4.5 0)
+			(at -4.535 2.25 0)
 			(layer "F.SilkS")
 			(effects
@@
 		(tags "resistor")
 		(property "Reference" "R5"
-			(at 0 -1.17 0)
+			(at -1.99 0 0)
 			(layer "F.SilkS")
 			(effects
@@
 		(tags "resistor")
 		(property "Reference" "R1"
-			(at 0 -1.17 -90)
+			(at -1.76 0 -90)
 			(layer "F.SilkS")
 			(effects
@@
 		(tags "mounting hole 4.3mm m4 iso14580")
 		(property "Reference" "H2"
-			(at 0 -4.5 0)
+			(at -4.535 -2.25 0)
 			(layer "F.SilkS")
 			(effects
@@
 		(at 122.38 93.11)
 		(property "Reference" "U1"
-			(at -6.715 -27.285 0)
+			(at -7.88 -26.36 0)
 			(layer "F.SilkS")
 			(effects
@@
 		(tags "mounting hole 4.3mm m4 iso14580")
 		(property "Reference" "H3"
-			(at 0 -4.5 0)
+			(at 4.5 2.25 0)
 			(layer "F.SilkS")
 			(effects
@@
 		(tags "resistor")
 		(property "Reference" "TH1"
-			(at 2.26 0.01 180)
+			(at -2.01 -0.01 180)
 			(layer "F.SilkS")
 			(effects
 				(font
-					(size 1 1)
-					(thickness 0.15)
+					(size 0.8 0.8)
+					(thickness 0.08)
 				)
 			)
@@
 		(tags "Through hole pin header THT 1x03 2.54mm single row")
 		(property "Reference" "J15"
-			(at 0 -2.33 90)
+			(at 0 7.475 90)
 			(layer "F.SilkS")
 			(effects
@@
 		(tags "mounting hole 4.3mm m4 iso14580")
 		(property "Reference" "H1"
-			(at 0 -4.5 0)
+			(at 4.5 -2.25 0)
 			(layer "F.SilkS")
 			(effects
@@
 		(tags "capacitor")
 		(property "Reference" "C12"
-			(at 0 -1.16 90)
+			(at -2.48 0 90)
 			(layer "F.SilkS")
 			(effects
 				(font
-					(size 1 1)
-					(thickness 0.15)
+					(size 0.8 0.8)
+					(thickness 0.08)
 				)
 			)
@@
 		(tags "Through hole pin header THT 1x02 2.54mm single row")
 		(property "Reference" "J5"
-			(at 0 -2.33 0)
+			(at 0 5.04 0)
 			(layer "F.SilkS")
 			(effects
@@
 		(tags "Through hole pin header THT 1x03 2.54mm single row")
 		(property "Reference" "J16"
-			(at 0 -2.33 90)
+			(at 0 7.5 90)
 			(layer "F.SilkS")
 			(effects
@@
 		(tags "capacitor")
 		(property "Reference" "C9"
-			(at 0 -1.16 90)
+			(at -1.98 0 90)
 			(layer "F.SilkS")
 			(effects
 				(font
-					(size 1 1)
-					(thickness 0.15)
+					(size 0.8 0.8)
+					(thickness 0.08)
 				)
 			)
@@
 		(tags "SOT TO_SOT_SMD")
 		(property "Reference" "U2"
-			(at 0 -2.4 0)
+			(at -2.5625 2.5 180)
 			(layer "F.SilkS")
 			(effects

Commit message: PCB edit
Routing:
- net /RA2/AN2/VREF-/CVREF: track 0.00 -> 5.56 mm
- net /RA0/AN0: track 0.00 -> 5.47 mm
- net /RA1/AN1: track 0.00 -> 5.35 mm
- net /*MCLR/VPP/RE3: track 3.28 -> 8.53 mm
Changed lines of the file:
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@@
+	)
+	(segment
+		(start 145.5925 68.985)
+		(end 146.7425 70.135)
+		(width 0.2)
+		(layer "In1.Cu")
+		(net 19)
+	)
+	(segment
+		(start 146.7425 70.135)
+		(end 150.365 70.135)
+		(width 0.2)
+		(layer "In1.Cu")
+		(net 19)
+	)
+	(segment
+		(start 146.8575 72.8)
+		(end 143.1 72.8)
+		(width 0.2)
+		(layer "F.Cu")
+		(net 20)
+	)
+	(segment
+		(start 148.1325 71.525)
+		(end 146.8575 72.8)
+		(width 0.2)
+		(layer "F.Cu")
+		(net 20)
+	)
+	(segment
+		(start 145.5925 71.525)
+		(end 146.8675 72.8)
+		(width 0.2)
+		(layer "In1.Cu")
+		(net 25)
+	)
+	(segment
+		(start 146.8675 72.8)
+		(end 150.415 72.8)
+		(width 0.2)
+		(layer "In1.Cu")
+		(net 25)
+	)
+	(segment
+		(start 146.9825 70.135)
+		(end 143.135 70.135)
+		(width 0.2)
+		(layer "F.Cu")
+		(net 38)
+	)
+	(segment
+		(start 148.1325 68.985)
+		(end 146.9825 70.135)
+		(width 0.2)
+		(layer "F.Cu")
+		(net 38)
 	)
 	(segment

Commit message: lots
Parts:
- moved J6 4.00 mm to (116.0, 122.0)
Routing:
- net /RB0/INT0/FLT0/AN12: track 0.00 -> 111.3 mm
- net /RB1/INT1/AN10: track 0.00 -> 109.9 mm
- net /RB2/INT2/AN8: track 0.00 -> 108.5 mm
- net /RB3/AN9/CCP2(1): track 0.00 -> 107.0 mm
- net /RB4/KBI0/AN11: track 0.00 -> 105.5 mm
- net /RB5/KBI1/PGM: track 0.00 -> 104.1 mm
- net /RB6/KBI2/PGC: track 0.00 -> 102.7 mm
- net /RB7/KBI3/PGD: track 0.00 -> 102.3 mm
- net /RD2/PSP2: track 0.00 -> 91.9 mm
- net /RD3/PSP3: track 0.00 -> 90.5 mm
- net /RC4/SDI/SDA: track 0.00 -> 89.0 mm
- net /RC5/SDO: track 0.00 -> 87.4 mm
- net /RD4/PSP4: track 0.00 -> 78.3 mm
- net /RD5/PSP5/P1B: track 0.00 -> 77.1 mm
- net /RD6/PSP6/P1C: track 0.00 -> 76.1 mm
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
Commit message: neat
Routing:
- net /RC1/T1OSI/CCP2(1): track 50.4 -> 53.1 mm
- net /RC2/CCP1/P1A: track 54.3 -> 51.9 mm
- net /OSC2/CLKO/RA6: track 68.3 -> 70.5 mm
- net /RD0/PSP0: track 57.7 -> 55.6 mm
- net /RC0/T1OSO/T13CKI: track 50.3 -> 48.2 mm
- net /OSC1/CLKI/RA7: track 79.7 -> 77.7 mm
- net /RC3/SCK/SCL: track 54.0 -> 56.0 mm
- net /RD1/PSP1: track 57.9 -> 56.4 mm
- net /RA3/AN3/VREF+: track 39.0 -> 37.9 mm
- net /RA4/T0CKI/C1OUT: track 39.6 -> 38.5 mm
- net /RA5/AN4/SS*/HLVDIN/C2OUT: track 40.0 -> 38.9 mm
- net /RE0/RD*/AN5: track 40.4 -> 39.4 mm
- net /RA0/AN0: track 37.3 -> 36.3 mm
- net /RE1/WR*/AN6: track 41.0 -> 40.0 mm
- net /RA1/AN1: track 37.8 -> 36.8 mm
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
Commit message: more routing
Routing:
- net GND: vias 13 -> 10
